Commit message: Added more services to wsg_50_sim_driver to fake real gripper services.

File: trunk/wsg_50_simulation/urdf/wsg_50.urdf.xacro (robot description, xacro)
@@ -1,24 +1,12 @@
 <?xml version="1.0"?>
 <robot name="wsg_50"
-       xmlns:xi="http://www.w3.org/2001/XInclude"
-       xmlns:gazebo="http://playerstage.sourceforge.net/gazebo/xmlschema/#gz"
-       xmlns:model="http://playerstage.sourceforge.net/gazebo/xmlschema/#model"
-       xmlns:sensor="http://playerstage.sourceforge.net/gazebo/xmlschema/#sensor"
-       xmlns:body="http://playerstage.sourceforge.net/gazebo/xmlschema/#body"
-       xmlns:geom="http://playerstage.sourceforge.net/gazebo/xmlschema/#geom"
-       xmlns:joint="http://playerstage.sourceforge.net/gazebo/xmlschema/#joint"
-       xmlns:interface="http://playerstage.sourceforge.net/gazebo/xmlschema/#interface"
-       xmlns:rendering="http://playerstage.sourceforge.net/gazebo/xmlschema/#rendering"
-       xmlns:renderable="http://playerstage.sourceforge.net/gazebo/xmlschema/#renderable"
-       xmlns:controller="http://playerstage.sourceforge.net/gazebo/xmlschema/#controller"
-       xmlns:physics="http://playerstage.sourceforge.net/gazebo/xmlschema/#physics"
-       xmlns:xacro="http://ros.org/wiki/xacro">
+	 xmlns:xacro="http://ros.org/wiki/xacro">
 <xacro:macro name="wsg_50_xacro" params="parent *origin">
- <joint name="arm_gripper_joint" type="fixed">
+ <joint name="anterior_gripper_joint" type="fixed">
     <insert_block name="origin"/>
     <parent link="${parent}"/>
     <child link="wsg_50_base_link"/>
  </joint>
- <!-- BASE LINK -->
+<!-- BASE LINK -->
  <link name="wsg_50_base_link">
       <inertial>
@@ -33,5 +21,5 @@
           <origin xyz="0.0 0 0" rpy="0 0 0" />
           <geometry>
-             <mesh filename="package://wsg_50_simulation/meshes/WSG50_110.stl" scale="0.001 0.001 0.001"/>
+             <mesh filename="package://wsg_50_simulation/meshes/WSG50_110.stl" scale="1 1 1"/>
 	     <!--box size="0.146 0.05 0.0735"/-->
           </geometry>
@@ -44,5 +32,5 @@
           <geometry>
 	     <!--box size="0.146 0.05 0.0735"/-->
-             <mesh filename="package://wsg_50_simulation/meshes/WSG50_110.stl" scale="0.001 0.001 0.001"/>
+             <mesh filename="package://wsg_50_simulation/meshes/WSG50_110.stl" scale="1 1 1"/>
          </geometry>
      </collision>
@@ -96,5 +84,5 @@
   <gazebo reference="gripper_left">
     <material>Gazebo/Blue</material>
-    <turnGravityOff>true</turnGravityOff>
+    <turnGravityOff>false</turnGravityOff>
   </gazebo>
   <!-- LEFT FINGER -->
@@ -133,5 +121,5 @@
   <gazebo reference="finger_left">
     <material>Gazebo/Blue</material>
-    <turnGravityOff>true</turnGravityOff>
+    <turnGravityOff>false</turnGravityOff>
   </gazebo>
   <!-- GRIPPER RIGHT -->
@@ -179,5 +167,5 @@
   <gazebo reference="gripper_right">
     <material>Gazebo/White</material>
-    <turnGravityOff>true</turnGravityOff>
+    <turnGravityOff>false</turnGravityOff>
   </gazebo>
   <!-- RIGHT FINGER -->
@@ -216,14 +204,6 @@
   <gazebo reference="finger_right">
     <material>Gazebo/White</material>
-    <turnGravityOff>true</turnGravityOff>
-  </gazebo>
-  <!-- PR2_ACTARRAY -->
-  <!--gazebo>
-     <controller:gazebo_ros_controller_manager name="gazebo_ros_controller_manager" plugin="libgazebo_ros_controller_manager.so">
-       <alwaysOn>true</alwaysOn>
-       <updateRate>1000.0</updateRate>
-       <interface:audio name="gazebo_ros_controller_manager_dummy_iface" />
-     </controller:gazebo_ros_controller_manager>
-  </gazebo-->
+    <turnGravityOff>false</turnGravityOff>
+  </gazebo>
 </xacro:macro>
 </robot>

Commit message: Updated URDF xacro fileand added new controllers and launch files to combine the gripper with the disponible arms.

File: trunk/wsg_50_simulation/urdf/wsg_50.urdf.xacro (robot description, xacro)
@@ -1,15 +1,18 @@
 <?xml version="1.0"?>
-<robot name="wsg_50"
-	 xmlns:xacro="http://ros.org/wiki/xacro">
-<xacro:macro name="wsg_50_xacro" params="parent *origin">
- <joint name="anterior_gripper_joint" type="fixed">
+<robot  xmlns:sensor="http://playerstage.sourceforge.net/gazebo/xmlschema/#sensor"
+	xmlns:controller="http://playerstage.sourceforge.net/gazebo/xmlschema/#controller"
+	xmlns:interface="http://playerstage.sourceforge.net/gazebo/xmlschema/#interface"
+        xmlns:xacro="http://ros.org/wiki/xacro"
+	name="wsg_50">
+<xacro:macro name="wsg_50_xacro" params="name parent *origin">
+ <joint name="${name}_anterior_gripper_joint" type="fixed">
     <insert_block name="origin"/>
     <parent link="${parent}"/>
-    <child link="wsg_50_base_link"/>
+    <child link="${name}_base_link"/>
  </joint>
 <!-- BASE LINK -->
- <link name="wsg_50_base_link">
-      <inertial>
-          <mass value="1.2" />
+ <link name="${name}_base_link">
+      <inertial>
+          <mass value="0.25" />
           <origin xyz="0 0 0" />
      	  <!--inertia ixx="1.0" ixy="0.0" ixz="0.0"
@@ -36,132 +39,135 @@
      </collision>
   </link>
-  <gazebo reference="wsg_50_base_link">
+  <gazebo reference="${name}_base_link">
     <material>Gazebo/Grey</material>
     <turnGravityOff>false</turnGravityOff>
   </gazebo>
   <!-- GRIPPER LEFT -->
-  <joint name="base_joint_gripper_left" type="prismatic">
+  <joint name="${name}_base_joint_gripper_left" type="prismatic">
      <limit lower="-0.055" upper="-0.0027" effort="1.0" velocity="1.0"/>
      <origin xyz="0 0 0" rpy="0 0 0" />      <!--origin xyz="-0.0067 0 0.049" rpy="0 0 0" /-->
-     <parent link="wsg_50_base_link"/>
-     <child link="gripper_left" />
+     <parent link="${name}_base_link"/>
+     <child link="${name}_gripper_left" />
      <dynamics friction="100" damping="100" />
      <axis xyz="1 0 0"/>
      <limit effort="100" velocity="100"/>
   </joint>
-  <transmission name="base_trans_left" type="pr2_mechanism_model/SimpleTransmission">
-     <actuator name="base_motor_left" />
-     <joint name="base_joint_gripper_left" />
+  <transmission name="${name}_base_trans_left" type="pr2_mechanism_model/SimpleTransmission">
+     <actuator name="${name}_base_motor_left" />
+     <joint name="${name}_base_joint_gripper_left" />
      <mechanicalReduction>1</mechanicalReduction>
      <motorTorqueConstant>1</motorTorqueConstant>
   </transmission>
-  <link name="gripper_left">
-      <inertial>
-          <mass value="0.1" />
-          <origin xyz="0 0 0" />
-      <inertia ixx="1.0" ixy="0.0" ixz="0.0"
-               iyy="1.0" iyz="0.0"
-               izz="1.0" />
-      </inertial>
-      <visual>
-          <origin xyz="0.0 0 0" rpy="0 0 0" />
-          <geometry>
-             <mesh filename="package://wsg_50_simulation/meshes/GUIDE_WSG50_110.stl" scale="0.001 0.001 0.001"/>
-	     <!--box size="0.0175 0.03 0.024"/-->
-          </geometry>
-          <material name="black">
-		<color rgba="0 0 0 0"/>
-      	  </material>
-      </visual>
-      <collision>
-          <origin xyz="0 0 0" rpy="0 0 0" />
-          <geometry>
-	     <!--box size="0.0175 0.03 0.024"/-->
-             <mesh filename="package://wsg_50_simulation/meshes/GUIDE_WSG50_110.stl" scale="0.001 0.001 0.001"/>
-         </geometry>
-     </collision>
-  </link>
-  <gazebo reference="gripper_left">
+  <link name="${name}_gripper_left">
+      <inertial>
+          <mass value="0.1" />
+          <origin xyz="0 0 0" />
+      <inertia ixx="1.0" ixy="0.0" ixz="0.0"
+               iyy="1.0" iyz="0.0"
+               izz="1.0" />
+      </inertial>
+      <visual>
+          <origin xyz="0.0 0 0" rpy="0 0 0" />
+          <geometry>
+             <mesh filename="package://wsg_50_simulation/meshes/GUIDE_WSG50_110.stl" scale="0.001 0.001 0.001"/>
+	     <!--box size="0.0175 0.03 0.024"/-->
+          </geometry>
+          <material name="black">
+		<color rgba="0 0 0 0"/>
+      	  </material>
+      </visual>
+      <collision>
+          <origin xyz="0 0 0" rpy="0 0 0" />
+          <geometry>
+	     <!--box size="0.0175 0.03 0.024"/-->
+             <mesh filename="package://wsg_50_simulation/meshes/GUIDE_WSG50_110.stl" scale="0.001 0.001 0.001"/>
+         </geometry>
+     </collision>
+     <contact_coefficients kd="1.0" kp="1000.0" mu="0"/>
+  </link>
+  <gazebo reference="${name}_gripper_left">
     <material>Gazebo/Blue</material>
     <turnGravityOff>false</turnGravityOff>
   </gazebo>
   <!-- LEFT FINGER -->
-  <joint name="guide_joint_finger_left" type="fixed">
+  <joint name="${name}_guide_joint_finger_left" type="fixed">
      <origin xyz="0 0 0.023" rpy="0 0 0" />
-     <parent link="gripper_left"/>
-     <child link="finger_left" />
+     <parent link="${name}_gripper_left"/>
+     <child link="${name}_finger_left" />
      <dynamics friction="100" damping="100" />
      <axis xyz="1 0 0"/>
      <limit effort="100" velocity="100"/>
   </joint>
-  <link name="finger_left">
-      <inertial>
-          <mass value="0.1" />
-          <origin xyz="0 0 0" />
-      <inertia ixx="1.0" ixy="0.0" ixz="0.0"
-               iyy="1.0" iyz="0.0"
-               izz="1.0" />
-      </inertial>
-      <visual>
-          <origin xyz="0.0 0 0" rpy="0 0 0" />
-          <geometry>
-             <mesh filename="package://wsg_50_simulation/meshes/WSG-FMF.stl" scale="0.001 0.001 0.001"/>
-          </geometry>
-          <material name="black">
-		<color rgba="0 0 0 0"/>
-      	  </material>
-      </visual>
-      <collision>
-          <origin xyz="0 0 0" rpy="0 0 0" />
-          <geometry>
-             <mesh filename="package://wsg_50_simulation/meshes/WSG-FMF.stl" scale="0.001 0.001 0.001"/>
-         </geometry>
-     </collision>
-  </link>
-  <gazebo reference="finger_left">
+  <link name="${name}_finger_left">
+      <inertial>
+          <mass value="0.1" />
+          <origin xyz="0 0 0" />
+      <inertia ixx="1.0" ixy="0.0" ixz="0.0"
+               iyy="1.0" iyz="0.0"
+               izz="1.0" />
+      </inertial>
+      <visual>
+          <origin xyz="0.0 0 0" rpy="0 0 0" />
+          <geometry>
+             <mesh filename="package://wsg_50_simulation/meshes/WSG-FMF.stl" scale="0.001 0.001 0.001"/>
+          </geometry>
+          <material name="black">
+		<color rgba="0 0 0 0"/>
+      	  </material>
+      </visual>
+      <collision>
+          <origin xyz="0 0 0" rpy="0 0 0" />
+          <geometry>
+             <mesh filename="package://wsg_50_simulation/meshes/WSG-FMF.stl" scale="0.001 0.001 0.001"/>
+         </geometry>
+     </collision>
+     <contact_coefficients kd="1.0" kp="1000.0" mu="0"/>
+  </link>
+  <gazebo reference="${name}_finger_left">
     <material>Gazebo/Blue</material>
     <turnGravityOff>false</turnGravityOff>
   </gazebo>
   <!-- GRIPPER RIGHT -->
-  <joint name="base_joint_gripper_right" type="prismatic">
+  <joint name="${name}_base_joint_gripper_right" type="prismatic">
      <limit lower="0.0027" upper="0.055" effort="1.0" velocity="1.0"/>
      <origin xyz="0 0 0" rpy="0 0 3.14159" />
-     <parent link="wsg_50_base_link"/>
-     <child link="gripper_right" />
+     <parent link="${name}_base_link"/>
+     <child link="${name}_gripper_right" />
      <axis xyz="-1 0 0"/>
      <dynamics friction="100" damping="100" />
      <limit effort="100" velocity="100"/>
   </joint>
-  <transmission name="base_trans_right" type="pr2_mechanism_model/SimpleTransmission">
-     <actuator name="base_motor_right" />
-     <joint name="base_joint_gripper_right" />
+  <transmission name="${name}_base_trans_right" type="pr2_mechanism_model/SimpleTransmission">
+     <actuator name="${name}_base_motor_right" />
+     <joint name="${name}_base_joint_gripper_right" />
      <mechanicalReduction>1</mechanicalReduction>
      <motorTorqueConstant>1</motorTorqueConstant>
   </transmission>
-    <link name="gripper_right">
-      <inertial>
-          <mass value="0.1" />
-          <origin xyz="0 0 0" />
-      <inertia ixx="1.0" ixy="0.0" ixz="0.0"
-               iyy="1.0" iyz="0.0"
-               izz="1.0" />
-      </inertial>
-      <visual>
-          <origin xyz="0.0 0 0" rpy="0 0 0" />
-          <geometry>
-             <mesh filename="package://wsg_50_simulation/meshes/GUIDE_WSG50_110.stl" scale="0.001 0.001 0.001"/>
-	     <!--box size="0.0175 0.03 0.024"/-->
-          </geometry>
-          <material name="black">
-		<color rgba="0 0 0 0"/>
-      	  </material>
-      </visual>
-      <collision>
-          <origin xyz="0 0 0" rpy="0 0 0" />
-          <geometry>
-	     <!--box size="0.0175 0.03 0.024"/-->
-             <mesh filename="package://wsg_50_simulation/meshes/GUIDE_WSG50_110.stl" scale="0.001 0.001 0.001"/>
-         </geometry>
-     </collision>
+    <link name="${name}_gripper_right">
+      <inertial>
+          <mass value="0.1" />
+          <origin xyz="0 0 0" />
+      <inertia ixx="1.0" ixy="0.0" ixz="0.0"
+               iyy="1.0" iyz="0.0"
+               izz="1.0" />
+      </inertial>
+      <visual>
+          <origin xyz="0.0 0 0" rpy="0 0 0" />
+          <geometry>
+             <mesh filename="package://wsg_50_simulation/meshes/GUIDE_WSG50_110.stl" scale="0.001 0.001 0.001"/>
+	     <!--box size="0.0175 0.03 0.024"/-->
+          </geometry>
+          <material name="black">
+		<color rgba="0 0 0 0"/>
+      	  </material>
+      </visual>
+      <collision>
+          <origin xyz="0 0 0" rpy="0 0 0" />
+          <geometry>
+	     <!--box size="0.0175 0.03 0.024"/-->
+             <mesh filename="package://wsg_50_simulation/meshes/GUIDE_WSG50_110.stl" scale="0.001 0.001 0.001"/>
+         </geometry>
+     </collision>
+     <contact_coefficients kd="1.0" kp="1000.0" mu="0"/>
   </link>
   <gazebo reference="gripper_right">
@@ -170,37 +176,38 @@
   </gazebo>
   <!-- RIGHT FINGER -->
-  <joint name="guide_joint_finger_right" type="fixed">
+  <joint name="${name}_guide_joint_finger_right" type="fixed">
      <origin xyz="0 0 0.023" rpy="0 0 0" />
-     <parent link="gripper_right"/>
-     <child link="finger_right" />
+     <parent link="${name}_gripper_right"/>
+     <child link="${name}_finger_right" />
      <dynamics friction="100" damping="100" />
      <axis xyz="1 0 0"/>
      <limit effort="100" velocity="100"/>
   </joint>
-  <link name="finger_right">
-      <inertial>
-          <mass value="0.1" />
-          <origin xyz="0 0 0" />
-      <inertia ixx="1.0" ixy="0.0" ixz="0.0"
-               iyy="1.0" iyz="0.0"
-               izz="1.0" />
-      </inertial>
-      <visual>
-          <origin xyz="0.0 0 0" rpy="0 0 0" />
-          <geometry>
-             <mesh filename="package://wsg_50_simulation/meshes/WSG-FMF.stl" scale="0.001 0.001 0.001"/>
-          </geometry>
-          <material name="black">
-		<color rgba="0 0 0 0"/>
-      	  </material>
-      </visual>
-      <collision>
-          <origin xyz="0 0 0" rpy="0 0 0" />
-          <geometry>
-             <mesh filename="package://wsg_50_simulation/meshes/WSG-FMF.stl" scale="0.001 0.001 0.001"/>
-         </geometry>
-     </collision>
-  </link>
-  <gazebo reference="finger_right">
+  <link name="${name}_finger_right">
+      <inertial>
+          <mass value="0.1" />
+          <origin xyz="0 0 0" />
+      <inertia ixx="1.0" ixy="0.0" ixz="0.0"
+               iyy="1.0" iyz="0.0"
+               izz="1.0" />
+      </inertial>
+      <visual>
+          <origin xyz="0.0 0 0" rpy="0 0 0" />
+          <geometry>
+             <mesh filename="package://wsg_50_simulation/meshes/WSG-FMF.stl" scale="0.001 0.001 0.001"/>
+          </geometry>
+          <material name="black">
+		<color rgba="0 0 0 0"/>
+      	  </material>
+      </visual>
+      <collision>
+          <origin xyz="0 0 0" rpy="0 0 0" />
+          <geometry>
+             <mesh filename="package://wsg_50_simulation/meshes/WSG-FMF.stl" scale="0.001 0.001 0.001"/>
+         </geometry>
+     </collision>
+     <contact_coefficients kd="1.0" kp="1000.0" mu="0"/>
+  </link>
+  <gazebo reference="${name}_finger_right">
     <material>Gazebo/White</material>
     <turnGravityOff>false</turnGravityOff>
